Commit message: Add Gazebo simulation with drive, depth camera and lidar

File: description/robot.urdf.xacro (robot description, xacro)
@@ -1,13 +1,212 @@
 <?xml version="1.0"?>
-<robot xmlns:xacro="http://www.ros.org/wiki/xacro"  name="robot">
-        <link name="base_link">
-        <visual>
-            <geometry>
-                <box size="0.3 0.2 0.1"/>
-            </geometry>
-            <material name="blue">
-                <color rgba="0.2 0.4 0.9 1"/>
-            </material>
-        </visual>
-    </link>
+<robot xmlns:xacro="http://www.ros.org/wiki/xacro" name="robot">
+    <material name="blue"><color rgba="0.2 0.4 0.9 1"/></material>
+    <material name="black"><color rgba="0.1 0.1 0.1 1"/></material>
+    <material name="red"><color rgba="0.9 0.2 0.2 1"/></material>
+    <material name="gray"><color rgba="0.6 0.6 0.6 1"/></material>
+    <!-- BODY -->
+    <link name="base_link">
+        <visual>
+            <origin xyz="0 0 0.05"/>
+            <geometry><box size="0.3 0.2 0.1"/></geometry>
+            <material name="blue"/>
+        </visual>
+        <collision>
+            <origin xyz="0 0 0.05"/>
+            <geometry><box size="0.3 0.2 0.1"/></geometry>
+        </collision>
+        <inertial>
+            <origin xyz="0 0 0.05"/>
+            <mass value="0.5"/>
+            <inertia ixx="0.002083" ixy="0" ixz="0" iyy="0.004167" iyz="0" izz="0.005417"/>
+        </inertial>
+    </link>
+    <!-- LEFT WHEEL -->
+    <joint name="left_wheel_joint" type="continuous">
+        <parent link="base_link"/>
+        <child link="left_wheel"/>
+        <origin xyz="0 0.12 0" rpy="-1.5708 0 0"/>
+        <axis xyz="0 0 1"/>
+    </joint>
+    <link name="left_wheel">
+        <visual>
+            <geometry><cylinder radius="0.05" length="0.04"/></geometry>
+            <material name="black"/>
+        </visual>
+        <collision>
+            <geometry><cylinder radius="0.05" length="0.04"/></geometry>
+        </collision>
+        <inertial>
+            <mass value="0.05"/>
+            <inertia ixx="0.0000379" ixy="0" ixz="0" iyy="0.0000379" iyz="0" izz="0.0000625"/>
+        </inertial>
+    </link>
+    <!-- RIGHT WHEEL -->
+    <joint name="right_wheel_joint" type="continuous">
+        <parent link="base_link"/>
+        <child link="right_wheel"/>
+        <origin xyz="0 -0.12 0" rpy="1.5708 0 0"/>
+        <axis xyz="0 0 -1"/>
+    </joint>
+    <link name="right_wheel">
+        <visual>
+            <geometry><cylinder radius="0.05" length="0.04"/></geometry>
+            <material name="black"/>
+        </visual>
+        <collision>
+            <geometry><cylinder radius="0.05" length="0.04"/></geometry>
+        </collision>
+        <inertial>
+            <mass value="0.05"/>
+            <inertia ixx="0.0000379" ixy="0" ixz="0" iyy="0.0000379" iyz="0" izz="0.0000625"/>
+        </inertial>
+    </link>
+    <!-- CASTER WHEEL -->
+    <joint name="caster_wheel_joint" type="fixed">
+        <parent link="base_link"/>
+        <child link="caster_wheel"/>
+        <origin xyz="0.12 0 -0.02"/>
+    </joint>
+    <link name="caster_wheel">
+        <visual>
+            <geometry><sphere radius="0.03"/></geometry>
+            <material name="gray"/>
+        </visual>
+        <collision>
+            <geometry><sphere radius="0.03"/></geometry>
+        </collision>
+        <inertial>
+            <mass value="0.02"/>
+            <inertia ixx="0.0000072" ixy="0" ixz="0" iyy="0.0000072" iyz="0" izz="0.0000072"/>
+        </inertial>
+    </link>
+    <!-- CAMERA -->
+    <joint name="camera_joint" type="fixed">
+        <parent link="base_link"/>
+        <child link="camera_link"/>
+        <origin xyz="0.12 0 0.115"/>
+    </joint>
+    <link name="camera_link">
+        <visual>
+            <geometry><box size="0.03 0.06 0.03"/></geometry>
+            <material name="red"/>
+        </visual>
+        <collision>
+            <geometry><box size="0.03 0.06 0.03"/></geometry>
+        </collision>
+        <inertial>
+            <mass value="0.02"/>
+            <inertia ixx="0.0000075" ixy="0" ixz="0" iyy="0.000003" iyz="0" izz="0.0000075"/>
+        </inertial>
+    </link>
+    <joint name="camera_optical_joint" type="fixed">
+        <parent link="camera_link"/>
+        <child link="camera_link_optical"/>
+        <origin xyz="0 0 0" rpy="-1.5707963 0 -1.5707963"/>
+    </joint>
+    <link name="camera_link_optical"></link>
+    <!-- GAZEBO COLOURS -->
+    <gazebo reference="base_link">
+        <material>Gazebo/Blue</material>
+    </gazebo>
+    <gazebo reference="left_wheel">
+        <material>Gazebo/Black</material>
+    </gazebo>
+    <gazebo reference="right_wheel">
+        <material>Gazebo/Black</material>
+    </gazebo>
+    <gazebo reference="caster_wheel">
+        <material>Gazebo/Grey</material>
+        <mu1 value="0.001"/>
+        <mu2 value="0.001"/>
+    </gazebo>
+    <!-- DRIVE PLUGIN -->
+    <gazebo>
+        <plugin name="diff_drive" filename="libgazebo_ros_diff_drive.so">
+            <left_joint>left_wheel_joint</left_joint>
+            <right_joint>right_wheel_joint</right_joint>
+            <wheel_separation>0.24</wheel_separation>
+            <wheel_diameter>0.1</wheel_diameter>
+            <max_wheel_torque>20</max_wheel_torque>
+            <max_wheel_acceleration>10.0</max_wheel_acceleration>
+            <odometry_frame>odom</odometry_frame>
+            <robot_base_frame>base_link</robot_base_frame>
+            <publish_odom>true</publish_odom>
+            <publish_odom_tf>true</publish_odom_tf>
+            <publish_wheel_tf>true</publish_wheel_tf>
+        </plugin>
+    </gazebo>
+    <!-- CAMERA SENSOR -->
+    <gazebo reference="camera_link">
+        <material>Gazebo/Red</material>
+        <sensor name="camera" type="depth">
+            <pose>0 0 0 0 0 0</pose>
+            <visualize>true</visualize>
+            <update_rate>10</update_rate>
+            <camera>
+                <horizontal_fov>1.089</horizontal_fov>
+                <image>
+                    <format>R8B8G8</format>
+                    <width>640</width>
+                    <height>480</height>
+                </image>
+                <clip>
+                    <near>0.05</near>
+                    <far>8.0</far>
+                </clip>
+            </camera>
+            <plugin name="camera_controller" filename="libgazebo_ros_camera.so">
+                <frame_name>camera_link_optical</frame_name>
+                <min_depth>0.1</min_depth>
+                <max_depth>8.0</max_depth>
+            </plugin>
+        </sensor>
+    </gazebo>
+    <!-- LIDAR -->
+    <joint name="laser_joint" type="fixed">
+        <parent link="base_link"/>
+        <child link="laser_frame"/>
+        <origin xyz="-0.05 0 0.14" rpy="0 0 0"/>
+    </joint>
+    <link name="laser_frame">
+        <visual>
+            <geometry><cylinder radius="0.03" length="0.08"/></geometry>
+            <material name="black"/>
+        </visual>
+        <collision>
+            <geometry><cylinder radius="0.03" length="0.08"/></geometry>
+        </collision>
+        <inertial>
+            <mass value="0.05"/>
+            <inertia ixx="0.0000300" ixy="0" ixz="0" iyy="0.0000300" iyz="0" izz="0.0000225"/>
+        </inertial>
+    </link>
+    <gazebo reference="laser_frame">
+        <material>Gazebo/Black</material>
+        <sensor name="laser" type="ray">
+            <pose>0 0 0 0 0 0</pose>
+            <visualize>false</visualize>
+            <update_rate>10</update_rate>
+            <ray>
+                <scan>
+                    <horizontal>
+                        <samples>360</samples>
+                        <min_angle>-3.14</min_angle>
+                        <max_angle>3.14</max_angle>
+                    </horizontal>
+                </scan>
+                <range>
+                    <min>0.3</min>
+                    <max>12</max>
+                </range>
+            </ray>
+            <plugin name="laser_controller" filename="libgazebo_ros_ray_sensor.so">
+                <ros>
+                    <argument>~/out:=scan</argument>
+                </ros>
+                <output_type>sensor_msgs/LaserScan</output_type>
+                <frame_name>laser_frame</frame_name>
+            </plugin>
+        </sensor>
+    </gazebo>
 </robot>
